File: DCC_Booster PCB/DCC_Booster.kicad_pcb (KiCad board)
At the start: 2 copper layers, 96 parts, among them J1 Conn_01x04, J2 4P4C, J3 4P4C, J4 Prog, J5 Jack-DC, Q1 Q_NMOS_GDS, Q2 Q_NMOS_GDS, Q3 Q_NMOS_GDS, Q4 Q_NMOS_GDS, SW1 SW_DIP_x05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

Commit message: worked on PCB
Parts:
- J2, J3: footprint Connector_RJ:RJ12_Amphenol_54601 -> SparkFun-Connectors:RJ9
- moved Q3 93.9 mm to (90.8, 83.4), turned to 90 degrees
- moved D12 87.7 mm to (99.7, 83.4), turned to 90 degrees
- moved D13 83.1 mm to (108.2, 83.4), turned to -90 degrees
- moved Q4 80.0 mm to (116.9, 83.4), turned to 90 degrees
- moved Q1 79.4 mm to (90.8, 96.1), turned to 90 degrees
- moved D10 72.0 mm to (99.7, 96.1), turned to 90 degrees
- moved R5 70.8 mm to (92.7, 109.2), turned to -90 degrees
- moved R4 70.7 mm to (90.2, 109.2), turned to -90 degrees
- moved C10 68.8 mm to (87.6, 108.6), turned to 90 degrees
- moved D8 68.1 mm to (85.1, 115.6), turned to -90 degrees
- moved R15 67.0 mm to (123.2, 98.4)
- moved D11 66.3 mm to (108.2, 96.1), turned to -90 degrees
- moved Q2 62.4 mm to (116.9, 96.1), turned to 90 degrees
- moved U4 60.8 mm to (90.8, 115.8), turned to 90 degrees
- moved C7 59.0 mm to (76.8, 123.2), turned to 180 degrees
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Routing:
- net GND: track 0.00 -> 340.5 mm
- net +24V: track 0.00 -> 110.5 mm
- net +15V: track 0.00 -> 87.9 mm
- net +5V: track 0.00 -> 69.0 mm, vias 0 -> 5
- net Net-(D1-Pad1): track 0.00 -> 59.2 mm, vias 0 -> 1
- net Net-(D2-Pad1): track 0.00 -> 46.6 mm
- net Net-(Q3-Pad1): track 0.00 -> 42.9 mm, vias 0 -> 2
- net Net-(U3-Pad11): track 0.00 -> 37.3 mm, vias 0 -> 2
- net Net-(U3-Pad8): track 0.00 -> 37.2 mm, vias 0 -> 2
- net Net-(C10-Pad2): track 0.00 -> 33.0 mm, vias 0 -> 2
- net Net-(U3-Pad3): track 0.00 -> 31.6 mm, vias 0 -> 2
- net Net-(U3-Pad6): track 0.00 -> 31.0 mm
- net Net-(C11-Pad2): track 0.00 -> 29.1 mm, vias 0 -> 2
- net Net-(Q2-Pad1): track 0.00 -> 29.1 mm, vias 0 -> 2
- net SYSLED: track 0.00 -> 28.6 mm
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
Commit message: pcb almost done
needs labels
Parts:
- added H1: MountingHole_3.2mm_M3, MountingHole:MountingHole_3.2mm_M3, F.Cu at (130.8, 133.3)
- added H2: MountingHole_3.2mm_M3, MountingHole:MountingHole_3.2mm_M3, F.Cu at (57.1, 133.3)
- added H3: MountingHole_3.2mm_M3, MountingHole:MountingHole_3.2mm_M3, F.Cu at (66.0, 57.1)
- moved R15 6.25 mm to (125.7, 92.7), turned to 0 degrees
- moved J5 2.14 mm to (47.0, 36.2)
- moved J2 1.27 mm to (40.6, 118.1)
- moved J3 1.27 mm to (40.6, 130.8)
Routing:
- net GND: track 340.5 -> 648.6 mm, vias 0 -> 14
- net +5V: track 69.0 -> 300.8 mm, vias 5 -> 10
- net +15V: track 87.9 -> 223.7 mm, vias 0 -> 24
- net Net-(C17-Pad1): track 3.39 -> 119.1 mm, vias 0 -> 1
- net Net-(D10-Pad2): track 15.9 -> 99.5 mm, vias 0 -> 2
- net Net-(D12-Pad2): track 24.7 -> 82.8 mm, vias 0 -> 2
- net DCC_Enable: track 20.5 -> 76.9 mm, vias 2 -> 3
- net DCC_POL: track 3.19 -> 50.9 mm, vias 0 -> 1
- net Drv_Status: track 0.00 -> 42.7 mm, vias 0 -> 2
- net DCC_Sig: track 0.00 -> 41.6 mm, vias 0 -> 2
- net TestMode: track 6.84 -> 40.4 mm, vias 0 -> 1
- net Net-(Q4-Pad1): track 28.1 -> 54.5 mm
- net Net-(R30-Pad2): track 0.00 -> 20.4 mm, vias 0 -> 2
- net VPP: track 0.00 -> 19.1 mm
- net Net-(C11-Pad2): track 29.1 -> 46.9 mm, vias 2 -> 0
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- added copper zone on B.Cu, net +15V
- added copper zone on B.Cu, net GND
Other:
- board outline added: 99.1 x 109.2 mm

Commit message: PCB ordered
Routing:
- net +15V: track 223.7 -> 210.8 mm
- net Net-(D10-Pad2): track 99.5 -> 98.9 mm, vias 2 -> 16
- net Net-(D13-Pad2): vias 0 -> 24
- net Net-(D12-Pad2): vias 2 -> 16
- net Net-(D11-Pad2): vias 0 -> 24
- added copper zone on B.Cu, net Net-(D10-Pad2)
- added copper zone on B.Cu, net Net-(D11-Pad2)
- added copper zone on B.Cu, net Net-(D12-Pad2)
- added copper zone on B.Cu, net Net-(D13-Pad2)
Other:
- rule pad_to_mask_clearance: 0.051 -> 0
- rule solder_mask_min_width: 0.25 -> 0.1016
- board text added: "+15V"
- board text added: "+24V"
- board text added: "+5V"
- board text added: "CSel0 CSel1 CSel2 N/R Test"
- board text added: "DCC Booster Rev. n/c"
- board text added: "DCC Sig OK"
- board text added: "DMFE 2019"
- board text added: "DRV"
- board text added: "PWR IN"
- board text added: "SYS LED"
