File: DCC_Booster Rev A PCB/DCC_Booster.sch (KiCad schematic (older format))
At the start: 96 parts, among them J1 Conn_01x04, J2 4P4C, J3 4P4C, J4 Prog, Q1 Q_NMOS_GDS, Q2 Q_NMOS_GDS, Q3 Q_NMOS_GDS, Q4 Q_NMOS_GDS, SW1 SW_DIP_x05, U1 MC34167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

Commit message: Schematic Rev A
Parts:
- added C19, C20, C21, C22: 0.1uf50v, Capacitor_SMD:C_0805_2012Metric_Pad1.15x1.40mm_HandSolder, symbol Device:C
- added D21, D22, D23, D24: 1N4148W, Diode_SMD:D_SOD-123, symbol Diode:1N4148W
- added D25, D26: BZT52C15, Diode_SMD:D_SOD-123, symbol Diode:BZT52Bxx
- added R35, R36: 10K, Resistor_SMD:R_0805_2012Metric_Pad1.15x1.40mm_HandSolder, symbol Device:R
- added R37, R38: 100, Resistor_SMD:R_0805_2012Metric_Pad1.15x1.40mm_HandSolder, symbol Device:R
- added TP1: GND, symbol Connector:TestPoint
- added TP2: +5V, symbol Connector:TestPoint
- added TP3: +24V, symbol Connector:TestPoint
- added TP4: +15V, symbol Connector:TestPoint
- added TP5: ISense, symbol Connector:TestPoint
- added U12, U13: LM555xM, Package_SO:SOIC-8_3.9x4.9mm_P1.27mm, symbol Timer:LM555xM
- C13: symbol Device:C -> Device:C_Small
- D8, D9: footprint Diode_SMD:D_SMA -> Diode_SMD:D_SOD-123
- gave numbers to parts that had none: 1
Connections:
- net labels added: C10N, C10P, C11N, C11P, GNDS
- wire segments 314 -> 377
- no-connect marks 2 -> 8
Other:
- moved on the sheet: C13, C17, R14, R30, R31, R32, R33

Commit message: Rev A PCB ordered
Parts:
- added C23, C24: 220uF, Capacitor_SMD:CP_Elec_10x10, symbol Device:CP1
- added D27: MRA4003T3G, Diode_SMD:D_SMA, symbol Diode:MRA4003T3G
- added TP6: DCC Sig, TestPoint:TestPoint_Pad_D2.0mm, symbol Connector:TestPoint
- D1, D10, D11, D12, D13, D2, D3, D4, D6, D7: footprint (none) -> Package_TO_SOT_SMD:TO-252-2
- D14: footprint Diode_THT:D_DO-35_SOD27_P7.62mm_Horizontal -> Diode_SMD:D_SOD-123
- D15, D16, D17, D18, D19, D20: footprint LED_THT:LED_D3.0mm_Horizontal_O1.27mm_Z2.0mm_Clear -> LED_THT:LED_D3.0mm
- FB1, FB2: footprint (none) -> Inductor_SMD:L_1812_4532Metric_Pad1.30x3.40mm_HandSolder
- J2, J3: footprint (none) -> SparkFun-Connectors:RJ9
- L1: footprint Inductor_THT:L_Radial_D24.4mm_P22.90mm_muRATA_1400series -> Inductor_THT:L_Radial_D24.4mm_P23.70mm_muRATA_1400series
- Q1, Q2, Q3, Q4: footprint Package_TO_SOT_SMD:TO-263-2 -> Package_TO_SOT_SMD:TO-252-2
- TP1, TP2, TP3, TP4, TP5: footprint (none) -> TestPoint:TestPoint_Pad_D2.0mm
- U11, U6, U9: footprint Package_TO_SOT_SMD:SOT-353_SC-70-5_Handsoldering -> Package_SO:TSOP-5_1.65x3.05mm_P0.95mm
- U12, U13: value LM555xM -> LM555CM
- U8: footprint Package_DIP:DIP-18_W7.62mm_LongPads -> Package_SO:SOIC-18W_7.5x11.6mm_P1.27mm
Connections:
- net labels added: Vdrive
- wire segments 377 -> 387
Other:
- note added: "15V"
- moved on the sheet: C2, D5

Commit message: Rev B
Parts:
- added C25, C26: 0.01uf50v, Capacitor_SMD:C_0805_2012Metric_Pad1.15x1.40mm_HandSolder, symbol Device:C_Small
Connections:
- wire segments 387 -> 401
Changed lines of the file:
@@
 Sheet 1 1
 Title "DCC Booster"
-Date "2020-03-05"
-Rev "A"
+Date "2020-03-11"
+Rev "B"
 Comp "DMFE"
 Comment1 "Model Railroad Digital Command Control Booster"
@@
 Connection ~ 7000 3150
 Connection ~ 7050 5750
+Connection ~ 7650 5100
+Connection ~ 7650 5250
 Connection ~ 7650 6150
 Connection ~ 8050 950
@@
 Connection ~ 9350 1600
 Connection ~ 9350 3350
+Connection ~ 9550 5100
+Connection ~ 9550 5250
 Connection ~ 9550 6150
 Connection ~ 9600 1600
@@
 Connection ~ 9700 3350
 Connection ~ 9900 3550
-Connection ~ 9900 4950
 Connection ~ 10000 3850
 Connection ~ 10150 5950
+Connection ~ 10300 5100
 Connection ~ 10300 5550
 NoConn ~ 1450 4750
@@
 	7150 5550 7100 5550
 Wire Wire Line
+	7600 5100 7650 5100
+Wire Wire Line
 	7700 1000 7700 950
 Wire Wire Line
@@
 	8100 2750 8100 2700
 Wire Wire Line
+	8250 5950 8250 6000
+Wire Wire Line
+	8250 6200 8250 6250
+Wire Wire Line
 	8400 2700 8450 2700
 Wire Wire Line
@@
 	9350 2950 9300 2950
 Wire Wire Line
+	9500 5100 9550 5100
+Wire Wire Line
 	9700 3350 9750 3350
 Wire Wire Line
 	10000 3850 10000 3900
 Wire Wire Line
+	10150 5950 10150 6000
+Wire Wire Line
+	10150 6200 10150 6250
+Wire Wire Line
 	10300 5550 10300 5500
 Wire Wire Line
@@
 	7800 3350 7700 3350
 Wire Wire Line
+	8000 6250 8000 6150
+Wire Wire Line
 	8250 5950 8150 5950
 Wire Wire Line
@@
 	9900 3850 10000 3850
 Wire Wire Line
-	9900 4850 9900 4950
-Wire Wire Line
-	9900 4950 9900 5050
+	9900 6250 9900 6150
 Wire Wire Line
 	10000 3850 10100 3850
@@
 	10150 5950 10050 5950
 Wire Wire Line
+	10300 5100 10300 5200
+Wire Wire Line
 	10300 5850 10300 5950
 Wire Wire Line
@@
 	7150 2250 7000 2250
 Wire Wire Line
+	7650 5100 7650 5250
+Wire Wire Line
 	8350 1300 8500 1300
 Wire Wire Line
@@
 	9150 4450 9300 4450
 Wire Wire Line
+	9550 5100 9550 5250
+Wire Wire Line
 	9750 1600 9600 1600
 Wire Wire Line
-	9750 4850 9900 4850
-Wire Wire Line
-	9900 5050 9750 5050
-Wire Wire Line
 	10300 5950 10150 5950
 Wire Wire Line
@@
 	7050 5750 7050 5950
 Wire Wire Line
+	7650 5100 7850 5100
+Wire Wire Line
 	8350 1800 8550 1800
 Wire Wire Line
@@
 	9250 1200 9050 1200
 Wire Wire Line
+	9550 5100 9750 5100
+Wire Wire Line
 	9700 3350 9700 3550
 Wire Wire Line
@@
 	8150 5550 8400 5550
 Wire Wire Line
+	8250 6250 8000 6250
+Wire Wire Line
 	8350 950  8350 1200
 Wire Wire Line
@@
 	9600 1600 9350 1600
 Wire Wire Line
+	10050 4800 10300 4800
+Wire Wire Line
+	10050 5100 10300 5100
+Wire Wire Line
 	10050 5550 10300 5550
 Wire Wire Line
-	10300 5200 10300 4950
+	10150 6250 9900 6250
 Wire Wire Line
 	1400 5400 1700 5400
@@
 	9150 4150 8850 4150
 Wire Wire Line
+	10300 4800 10300 5100
+Wire Wire Line
 	650  2900 1000 2900
 Wire Wire Line
@@
 	7750 3750 8100 3750
 Wire Wire Line
+	8000 6150 7650 6150
+Wire Wire Line
 	8100 2700 7750 2700
 Wire Wire Line
@@
 	9050 1700 8700 1700
 Wire Wire Line
+	9900 6150 9550 6150
+Wire Wire Line
 	1450 4150 1850 4150
 Wire Wire Line
@@
 	8550 3550 8550 3950
 Wire Wire Line
-	10300 4950 9900 4950
-Wire Wire Line
 	1400 6200 1400 6650
 Wire Wire Line
@@
 	7650 5250 7050 5250
 Wire Wire Line
-	9550 5250 8950 5250
+	8950 5250 9550 5250
 Wire Wire Line
 	4050 1150 4050 1800
@@
 Text GLabel 6900 1400 0    50   Input ~ 0
 DCC_Enable
+Text GLabel 7600 5100 0    50   Input ~ 0
+C10N
 Text GLabel 7850 4800 0    50   Input ~ 0
 C10P
-Text GLabel 7850 5100 0    50   Input ~ 0
-C10N
 Text GLabel 8700 1200 2    50   Input ~ 0
 C10P
@@
 Text GLabel 8700 3350 0    50   Input ~ 0
 C11N
-Text GLabel 9450 4850 0    50   Input ~ 0
+Text GLabel 9500 5100 0    50   Input ~ 0
+C11N
+Text GLabel 9750 4800 0    50   Input ~ 0
 C11P
-Text GLabel 9450 5050 0    50   Input ~ 0
-C11N
 Text GLabel 10050 1600 2    50   Input ~ 0
 NorthRail
@@
 $EndComp
 $Comp
+L Device:C_Small C25
+U 1 1 5E698CFB
+P 8250 6100
+F 0 "C25" H 8200 6200 50  0000 R CNN
+F 1 "0.01uf50v" H 8050 5850 50  0000 L CNN
+F 2 "Capacitor_SMD:C_0805_2012Metric_Pad1.15x1.40mm_HandSolder" H 8288 5950 50  0001 C CNN
+F 3 "~" H 8250 6100 50  0001 C CNN
+	1    8250 6100
+	1    0    0    -1
+$EndComp
+$Comp
+L Device:C_Small C26
+U 1 1 5E699F1F
+P 10150 6100
+F 0 "C26" H 10100 6200 50  0000 R CNN
+F 1 "0.01uf50v" H 9950 5850 50  0000 L CNN
+F 2 "Capacitor_SMD:C_0805_2012Metric_Pad1.15x1.40mm_HandSolder" H 10188 5950 50  0001 C CNN
+F 3 "~" H 10150 6100 50  0001 C CNN
+	1    10150 6100
+	1    0    0    -1
+$EndComp
+$Comp
 L Diode:MRA4003T3G D5
 U 1 1 5DC1301D
@@
 L Diode:1N4148W D22
 U 1 1 5E637F2B
-P 9600 4850
-F 0 "D22" H 9750 4900 50  0000 C CNN
-F 1 "1N4148W" V 9645 4930 50  0001 L CNN
-F 2 "Diode_SMD:D_SOD-123" H 9600 4675 50  0001 C CNN
-F 3 "https://www.vishay.com/docs/85748/1n4148w.pdf" H 9600 4850 50  0001 C CNN
-	1    9600 4850
+P 9900 4800
+F 0 "D22" H 10050 4850 50  0000 C CNN
+F 1 "1N4148W" V 9945 4880 50  0001 L CNN
+F 2 "Diode_SMD:D_SOD-123" H 9900 4625 50  0001 C CNN
+F 3 "https://www.vishay.com/docs/85748/1n4148w.pdf" H 9900 4800 50  0001 C CNN
+	1    9900 4800
 	1    0    0    -1
 $EndComp
@@
 L Diode:1N4148W D23
 U 1 1 5E639E88
-P 9600 5050
-F 0 "D23" H 9450 5000 50  0000 C CNN
-F 1 "1N4148W" V 9645 5130 50  0001 L CNN
-F 2 "Diode_SMD:D_SOD-123" H 9600 4875 50  0001 C CNN
-F 3 "https://www.vishay.com/docs/85748/1n4148w.pdf" H 9600 5050 50  0001 C CNN
-	1    9600 5050
+P 9900 5100
+F 0 "D23" H 9750 5050 50  0000 C CNN
+F 1 "1N4148W" V 9945 5180 50  0001 L CNN
+F 2 "Diode_SMD:D_SOD-123" H 9900 4925 50  0001 C CNN
+F 3 "https://www.vishay.com/docs/85748/1n4148w.pdf" H 9900 5100 50  0001 C CNN
+	1    9900 5100
 	-1   0    0    1
 $EndComp

Commit message: Rev B
Parts:
- added R39, R40: 10R, Resistor_SMD:R_0805_2012Metric_Pad1.15x1.40mm_HandSolder, symbol Device:R
Connections:
- wire segments 401 -> 411
Changed lines of the file:
@@
 Sheet 1 1
 Title "DCC Booster"
-Date "2020-03-11"
+Date "2020-05-08"
 Rev "B"
 Comp "DMFE"
@@
 Connection ~ 7650 5250
 Connection ~ 7650 6150
-Connection ~ 8050 950
+Connection ~ 7700 800
+Connection ~ 7700 950
+Connection ~ 7750 2550
+Connection ~ 7750 2700
 Connection ~ 8050 2000
-Connection ~ 8100 2700
 Connection ~ 8100 3750
 Connection ~ 8250 5950
-Connection ~ 8350 1200
 Connection ~ 8400 5100
 Connection ~ 8400 5550
-Connection ~ 8450 2950
+Connection ~ 8650 1200
+Connection ~ 8650 2950
+Connection ~ 8700 1200
+Connection ~ 8700 1600
 Connection ~ 8700 1700
+Connection ~ 8700 2950
+Connection ~ 8700 3350
 Connection ~ 8700 3450
 Connection ~ 8850 5750
@@
 	6000 950  6050 950
 Wire Wire Line
+	6000 1350 6000 1400
+Wire Wire Line
 	6000 1350 6000 1300
 Wire Wire Line
-	6000 1350 6000 1400
-Wire Wire Line
 	6000 3300 6000 3250
 Wire Wire Line
@@
 	7700 1000 7700 950
 Wire Wire Line
+	7750 2500 7750 2550
+Wire Wire Line
 	7750 2700 7750 2750
 Wire Wire Line
-	8050 900  8050 950
-Wire Wire Line
 	8050 1000 8050 950
 Wire Wire Line
-	8100 2650 8100 2700
-Wire Wire Line
 	8100 2750 8100 2700
 Wire Wire Line
@@
 	8250 6200 8250 6250
 Wire Wire Line
-	8400 2700 8450 2700
-Wire Wire Line
-	8400 2950 8450 2950
-Wire Wire Line
 	8400 5550 8400 5500
 Wire Wire Line
+	8600 800  8650 800
+Wire Wire Line
+	8600 2550 8650 2550
+Wire Wire Line
+	8650 1200 8700 1200
+Wire Wire Line
+	8650 1600 8700 1600
+Wire Wire Line
+	8650 2950 8700 2950
+Wire Wire Line
+	8650 3350 8700 3350
+Wire Wire Line
 	8650 6250 8650 6200
 Wire Wire Line
+	8700 1200 8750 1200
+Wire Wire Line
+	8700 2950 8750 2950
+Wire Wire Line
 	8850 4150 8850 4200
 Wire Wire Line
@@
 	7650 5350 7650 5250
 Wire Wire Line
+	7700 700  7700 800
+Wire Wire Line
 	7700 3250 7800 3250
 Wire Wire Line
@@
 	7650 5100 7650 5250
 Wire Wire Line
+	7700 800  7700 950
+Wire Wire Line
+	7750 2550 7750 2700
+Wire Wire Line
 	8350 1300 8500 1300
 Wire Wire Line
@@
 	7700 3350 7700 3600
 Wire Wire Line
+	7750 2550 8000 2550
+Wire Wire Line
 	8150 4800 8400 4800
 Wire Wire Line
@@
 	8250 6250 8000 6250
 Wire Wire Line
-	8350 950  8350 1200
-Wire Wire Line
-	8450 2700 8450 2950
-Wire Wire Line
-	8450 2950 8700 2950
+	8400 2950 8650 2950
 Wire Wire Line
 	9000 5550 9000 5300
@@
 	6350 1950 6350 2250
 Wire Wire Line
+	7700 800  8000 800
+Wire Wire Line
+	8350 1200 8650 1200
+Wire Wire Line
 	8400 3450 8700 3450
 Wire Wire Line
@@
 	8100 2700 7750 2700
 Wire Wire Line
-	8350 1200 8700 1200
-Wire Wire Line
 	8350 1700 8700 1700
 Wire Wire Line
@@
 	8550 3550 8550 3950
 Wire Wire Line
+	8650 800  8650 1200
+Wire Wire Line
+	8650 2550 8650 2950
+Wire Wire Line
 	1400 6200 1400 6650
 Wire Wire Line
@@
 	1850 4150 1850 4650
 Wire Wire Line
+	2000 2900 1500 2900
+Wire Wire Line
 	2000 2900 2500 2900
-Wire Wire Line
-	2000 2900 1500 2900
 Wire Wire Line
 	7000 1750 7000 2250
@@
 Text GLabel 7850 4800 0    50   Input ~ 0
 C10P
-Text GLabel 8700 1200 2    50   Input ~ 0
+Text GLabel 8650 1600 0    50   Input ~ 0
+C10N
+Text GLabel 8650 3350 0    50   Input ~ 0
+C11N
+Text GLabel 8750 1200 2    50   Input ~ 0
 C10P
-Text GLabel 8700 1600 0    50   Input ~ 0
-C10N
-Text GLabel 8700 2950 2    50   Input ~ 0
+Text GLabel 8750 2950 2    50   Input ~ 0
 C11P
-Text GLabel 8700 3350 0    50   Input ~ 0
-C11N
 Text GLabel 9500 5100 0    50   Input ~ 0
 C11N
@@
 L power:Vdrive #PWR014
 U 1 1 5E6484D3
-P 8050 900
-F 0 "#PWR014" H 7850 750 50  0001 C CNN
-F 1 "Vdrive" H 8065 1073 50  0000 C CNN
-F 2 "" H 8050 900 50  0001 C CNN
-F 3 "" H 8050 900 50  0001 C CNN
-	1    8050 900
+P 7700 700
+F 0 "#PWR014" H 7500 550 50  0001 C CNN
+F 1 "Vdrive" H 7715 873 50  0000 C CNN
+F 2 "" H 7700 700 50  0001 C CNN
+F 3 "" H 7700 700 50  0001 C CNN
+	1    7700 700
 	1    0    0    -1
 $EndComp
@@
 L power:Vdrive #PWR055
 U 1 1 5E647FED
-P 8100 2650
-F 0 "#PWR055" H 7900 2500 50  0001 C CNN
-F 1 "Vdrive" H 8115 2823 50  0000 C CNN
-F 2 "" H 8100 2650 50  0001 C CNN
-F 3 "" H 8100 2650 50  0001 C CNN
-	1    8100 2650
+P 7750 2500
+F 0 "#PWR055" H 7550 2350 50  0001 C CNN
+F 1 "Vdrive" H 7765 2673 50  0000 C CNN
+F 2 "" H 7750 2500 50  0001 C CNN
+F 3 "" H 7750 2500 50  0001 C CNN
+	1    7750 2500
 	1    0    0    -1
 $EndComp
@@
 $EndComp
 $Comp
+L Device:R R39
+U 1 1 5EB60E7C
+P 8450 800
+F 0 "R39" V 8350 800 50  0000 R CNN
+F 1 "10R" V 8450 850 50  0000 R CNN
+F 2 "Resistor_SMD:R_0805_2012Metric_Pad1.15x1.40mm_HandSolder" V 8380 800 50  0001 C CNN
+F 3 "~" H 8450 800 50  0001 C CNN
+	1    8450 800
+	0    1    1    0
+$EndComp
+$Comp
+L Device:R R40
+U 1 1 5EB618EF
+P 8450 2550
+F 0 "R40" V 8350 2550 50  0000 R CNN
+F 1 "10R" V 8450 2600 50  0000 R CNN
+F 2 "Resistor_SMD:R_0805_2012Metric_Pad1.15x1.40mm_HandSolder" V 8380 2550 50  0001 C CNN
+F 3 "~" H 8450 2550 50  0001 C CNN
+	1    8450 2550
+	0    1    1    0
+$EndComp
+$Comp
 L Device:R R4
 U 1 1 5DC392D2
@@
 L Diode:B140-E3 D8
 U 1 1 5DC40A05
-P 8200 950
-F 0 "D8" H 8200 850 50  0000 C CNN
-F 1 "B140-E3" H 8200 825 50  0001 C CNN
-F 2 "Diode_SMD:D_SOD-123" H 8200 775 50  0001 C CNN
-F 3 "http://www.vishay.com/docs/88946/b120.pdf" H 8200 950 50  0001 C CNN
-	1    8200 950
+P 8150 800
+F 0 "D8" H 8150 700 50  0000 C CNN
+F 1 "B140-E3" H 8150 675 50  0001 C CNN
+F 2 "Diode_SMD:D_SOD-123" H 8150 625 50  0001 C CNN
+F 3 "http://www.vishay.com/docs/88946/b120.pdf" H 8150 800 50  0001 C CNN
+	1    8150 800
 	-1   0    0    1
 $EndComp
@@
 L Diode:B140-E3 D9
 U 1 1 5DC4BA8D
-P 8250 2700
-F 0 "D9" H 8250 2600 50  0000 C CNN
-F 1 "B140-E3" H 8250 2575 50  0001 C CNN
-F 2 "Diode_SMD:D_SOD-123" H 8250 2525 50  0001 C CNN
-F 3 "http://www.vishay.com/docs/88946/b120.pdf" H 8250 2700 50  0001 C CNN
-	1    8250 2700
+P 8150 2550
+F 0 "D9" H 8150 2450 50  0000 C CNN
+F 1 "B140-E3" H 8150 2425 50  0001 C CNN
+F 2 "Diode_SMD:D_SOD-123" H 8150 2375 50  0001 C CNN
+F 3 "http://www.vishay.com/docs/88946/b120.pdf" H 8150 2550 50  0001 C CNN
+	1    8150 2550
 	-1   0    0    1
 $EndComp
