File: DCC_Booster Rev B PCB/DCC_Booster.sch (KiCad schematic (older format))
At the start: 125 parts, among them J1 Conn_01x04, J2 4P4C, J3 4P4C, J4 Prog, Q1 Q_NMOS_GDS, Q2 Q_NMOS_GDS, Q3 Q_NMOS_GDS, Q4 Q_NMOS_GDS, SW1 SW_DIP_x05, U1 MC34167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

Commit message: Rev B PCB
Parts:
- C17: value 0.1uf50v -> 1.0uf25v
- gave numbers to parts that had none: 2
Changed lines of the file:
@@
 	6000 950  6050 950
 Wire Wire Line
+	6000 1350 6000 1300
+Wire Wire Line
 	6000 1350 6000 1400
-Wire Wire Line
-	6000 1350 6000 1300
 Wire Wire Line
 	6000 3300 6000 3250
@@
 $EndComp
 $Comp
-L Device:R R?
+L Device:R R39
 U 1 1 5EB60E7C
 P 8450 800
-F 0 "R?" V 8350 800 50  0000 R CNN
+F 0 "R39" V 8350 800 50  0000 R CNN
 F 1 "10R" V 8450 850 50  0000 R CNN
 F 2 "Resistor_SMD:R_0805_2012Metric_Pad1.15x1.40mm_HandSolder" V 8380 800 50  0001 C CNN
@@
 $EndComp
 $Comp
-L Device:R R?
+L Device:R R40
 U 1 1 5EB618EF
 P 8450 2550
-F 0 "R?" V 8350 2550 50  0000 R CNN
+F 0 "R40" V 8350 2550 50  0000 R CNN
 F 1 "10R" V 8450 2600 50  0000 R CNN
 F 2 "Resistor_SMD:R_0805_2012Metric_Pad1.15x1.40mm_HandSolder" V 8380 2550 50  0001 C CNN
@@
 P 4950 3300
 F 0 "C17" H 5150 3200 50  0000 R CNN
-F 1 "0.1uf50v" H 5065 3255 50  0001 L CNN
+F 1 "1.0uf25v" H 4600 3200 50  0000 L CNN
 F 2 "Capacitor_SMD:C_0805_2012Metric_Pad1.15x1.40mm_HandSolder" H 4988 3150 50  0001 C CNN
 F 3 "~" H 4950 3300 50  0001 C CNN
